File: Circuit/esp-lvl.kicad_pcb (KiCad board)
At the start: 2 copper layers, 32 x 19 mm, 12 parts, among them J1 CONN_01X04, J2 CONN_01X04, J3 CONN_01X06, U1 MIC5205-3.3YM5, U2 ESP-12F

Commit message: v2
Parts:
- removed C2: 1u, Capacitor_SMD:C_0603_1608Metric_Pad1.05x0.95mm_HandSolder
- removed the R4 at (110.0, 78.0)
- removed the U1 at (111.3, 70.0)
- added D1: BAT54S, Package_TO_SOT_SMD:SOT-23, F.Cu at (158.8, 91.3)
- added D2: BAT54S, Package_TO_SOT_SMD:SOT-23, F.Cu at (162.6, 91.3)
- added D3: BAT54S, Package_TO_SOT_SMD:SOT-23, B.Cu at (145.1, 100.7)
- added G***: LOGO, LOGO, B.Cu at (159.8, 92.3)
- added J4: ESP_prog, Connectors:Tag-Connect_TC2030-IDC-NL, F.Cu at (135.5, 89.9)
- added R1: 10k, Resistor_SMD:R_0603_1608Metric, B.Cu at (146.8, 91.8)
- added R10: 2k2, Resistor_SMD:R_0603_1608Metric, F.Cu at (162.3, 99.8)
- added R2: 10k, Resistor_SMD:R_0603_1608Metric, B.Cu at (146.8, 90.0)
- added R6: R, Resistor_SMD:R_0603_1608Metric, F.Cu at (158.8, 97.8)
- added R8: R, Resistor_SMD:R_0603_1608Metric, F.Cu at (162.3, 97.8)
- added R9: R, Resistor_SMD:R_0603_1608Metric, B.Cu at (148.5, 100.5)
- added kibuzzard-6485947F: G***, kibuzzard-6485947F, F.Cu at (139.3, 102.3)
- added kibuzzard-64859500: G***, kibuzzard-64859500, F.Cu at (141.9, 102.3)
- added kibuzzard-64859500: G***, kibuzzard-64859500, F.Cu at (151.9, 102.3)
- added kibuzzard-64859549: G***, kibuzzard-64859549, F.Cu at (144.5, 102.3)
- added kibuzzard-64859551: G***, kibuzzard-64859551, F.Cu at (147.1, 102.3)
- added kibuzzard-64859557: G***, kibuzzard-64859557, F.Cu at (149.5, 102.3)
- added kibuzzard-64859561: G***, kibuzzard-64859561, F.Cu at (154.5, 102.3)
- added kibuzzard-64859916: G***, kibuzzard-64859916, F.Cu at (137.0, 94.6)
- added kibuzzard-64859921: G***, kibuzzard-64859921, F.Cu at (137.0, 100.6)
- added kibuzzard-64859928: G***, kibuzzard-64859928, F.Cu at (137.0, 103.1)
- added kibuzzard-6485998B: G***, kibuzzard-6485998B, F.Cu at (137.0, 97.5)
- added kibuzzard-648599E7: G***, kibuzzard-648599E7, F.Cu at (162.6, 95.2)
- added kibuzzard-64859B50: G***, kibuzzard-64859B50, F.Cu at (162.3, 103.0)
- added kibuzzard-6485D4C1: G***, kibuzzard-6485D4C1, B.Cu at (159.8, 99.3)
- added kibuzzard-6485EB90: G***, kibuzzard-6485EB90, F.Cu at (160.4, 87.6)
- added kibuzzard-64860007: G***, kibuzzard-64860007, F.Cu at (160.2, 105.2)
- C1: value 1u -> 100n; footprint Capacitor_SMD:C_0603_1608Metric_Pad1.05x0.95mm_HandSolder -> Capacitor_SMD:C_0603_1608Metric; moved to B.Cu
- J3: value CONN_01X06 -> CONN_01X07; footprint Connector_PinHeader_2.54mm:PinHeader_1x06_P2.54mm_Vertical -> Connector_PinHeader_2.54mm:PinHeader_1x07_P2.54mm_Vertical
- R3: renamed from R1; value 2k2 -> 10k; footprint passive:R_0603 -> Resistor_SMD:R_0603_1608Metric
- R4: renamed from R5; value 2k2 -> 10k; footprint passive:R_0603 -> Resistor_SMD:R_0603_1608Metric
- R5: renamed from R2; value 2k2 -> 10k; footprint passive:R_0603 -> Resistor_SMD:R_0603_1608Metric
- R7: renamed from R3; footprint passive:R_0603 -> Resistor_SMD:R_0603_1608Metric
- moved J1 53.3 mm to (135.3, 95.3)
- moved J2 53.3 mm to (159.3, 95.3)
- moved R3 53.3 mm to (146.8, 93.8)
- moved R4 53.3 mm to (146.8, 97.8)
- moved R5 53.3 mm to (146.8, 95.8)
- moved U1 53.3 mm to (146.8, 89.3)
- moved R7 52.7 mm to (158.8, 99.8), turned to 180 degrees
- moved J3 51.9 mm to (139.3, 104.0)
- moved C1 43.0 mm to (138.3, 100.8)
- renumbered U2 to U1
Connections:
- net Net-(R1-Pad1) renamed /GPIO0
- C1 pad 1: +5V -> +3V3
- J1 pad 3: +5V -> +3V3
- J3 pad 2: /SENS -> +3V3
- J3 pad 3: +5V -> /SENS
- J3 pad 4: +3V3 -> /SDA
- J3 pad 6: /SDA -> +3V3
- U1 pad 1: unconnected-(U2-Pad1) -> /RST
- U1 pad 19: /SDA -> /SDA_esp
- U1 pad 20: /SCL -> /SCL_esp
- U1 pad 21: unconnected-(U2-Pad21) -> /RX
- U1 pad 22: unconnected-(U2-Pad22) -> /TX
- U1 pad 3: +3V3 -> Net-(U1-EN)
- U1 pad 7: /SENS -> /SENS_esp
Routing:
- net +5V: track 58.7 -> 0.00 mm
- net /RST: track 0.00 -> 24.0 mm, vias 0 -> 2
- net /GPIO0: track 6.85 -> 27.8 mm, vias 1 -> 3
- net /RX: track 0.00 -> 19.8 mm
- net /TX: track 0.00 -> 19.5 mm
- net /SCL_esp: track 0.00 -> 16.8 mm
- net /SDA_esp: track 0.00 -> 12.5 mm
- net /SENS_esp: track 0.00 -> 10.5 mm, vias 0 -> 1
- net Net-(U1-EN): track 0.00 -> 7.39 mm, vias 0 -> 1
- net GND: track 29.1 -> 22.8 mm, vias 3 -> 4
- net /SCL: track 22.7 -> 17.4 mm, vias 1 -> 0
- net +3V3: track 84.2 -> 78.9 mm, vias 2 -> 15
- net /PWM_Bright: track 9.36 -> 5.46 mm, vias 1 -> 0
- net /SENS: track 10.0 -> 7.67 mm, vias 2 -> 0
- net /SDA: track 19.2 -> 17.8 mm, vias 1 -> 0
- added copper zone on B.Cu, net +3V3
Other:
- board size 32 x 19 mm -> 32 x 21.5 mm
- board text removed: "2022-06-06 Rev.1"
- board text removed: "3V3"
- board text removed: "5V"
- board text removed: "Colour"
- board text removed: "GND"
- board text removed: "LVL LED Light"
- board text removed: "NC Bright +5V GND"
- board text removed: "SCL"
- board text removed: "SDA"
- board text removed: "Sens"

Commit message: BOM updated
Parts:
- R6, R8, R9: value R -> 220R
Changed lines of the file:
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@@
         (effects (font (size 0.7 0.7) (thickness 0.15)))
     )
-    (fp_text value "R" (at 0 1.43 180) (layer "F.Fab")
+    (fp_text value "220R" (at 0 1.43 180) (layer "F.Fab")
         (effects (font (size 1 1) (thickness 0.15)))
     )
@@
         (effects (font (size 0.7 0.7) (thickness 0.15)))
     )
-    (fp_text value "R" (at 0 1.43) (layer "F.Fab")
+    (fp_text value "220R" (at 0 1.43) (layer "F.Fab")
         (effects (font (size 1 1) (thickness 0.15)))
     )
@@
         (effects (font (size 0.7 0.7) (thickness 0.15)) (justify mirror))
     )
-    (fp_text value "R" (at 0 -1.43 180) (layer "B.Fab")
+    (fp_text value "220R" (at 0 -1.43 180) (layer "B.Fab")
         (effects (font (size 1 1) (thickness 0.15)) (justify mirror))
     )
