File: Circuit/esp-lvl.kicad_sch (KiCad schematic)
At the start: 12 parts, among them J1 CONN_01X04, J2 CONN_01X04, J3 CONN_01X06, U1 MIC5205-3.3YM5, U2 ESP-12F

Commit message: v2
Parts:
- removed C1, C2: 1u, Capacitor_SMD:C_0603_1608Metric_Pad1.05x0.95mm_HandSolder, symbol passive:C
- removed J3: CONN_01X06, Connector_PinHeader_2.54mm:PinHeader_1x06_P2.54mm_Vertical, symbol connectors:CONN_01X06
- removed R4: 2k2, passive:R_0603, symbol resistors_0603:10k
- removed U1: MIC5205-3.3YM5, TO_SOT_Packages_SMD:SOT-23-5, symbol IC:MIC5205-3.3YM5
- added C1: 100n, Capacitor_SMD:C_0603_1608Metric, symbol Device:C
- added D1, D2, D3: BAT54S, Package_TO_SOT_SMD:SOT-23, symbol diode_fast:BAT54S
- added J3: CONN_01X07, Connector_PinHeader_2.54mm:PinHeader_1x07_P2.54mm_Vertical, symbol connectors:CONN_01X07
- added J4: ESP_prog, Connectors:Tag-Connect_TC2030-IDC-NL, symbol others:ESP_prog
- added R1, R2: 10k, Resistor_SMD:R_0603_1608Metric, symbol Device:R
- added R10: 2k2, Resistor_SMD:R_0603_1608Metric, symbol resistors_0603:10k
- added R6, R8, R9: R, Resistor_SMD:R_0603_1608Metric, symbol Device:R
- R3: renamed from R1; value 2k2 -> 10k; footprint passive:R_0603 -> Resistor_SMD:R_0603_1608Metric
- R4: renamed from R5; value 2k2 -> 10k; footprint passive:R_0603 -> Resistor_SMD:R_0603_1608Metric
- R5: renamed from R2; value 2k2 -> 10k; footprint passive:R_0603 -> Resistor_SMD:R_0603_1608Metric
- R7: renamed from R3; footprint passive:R_0603 -> Resistor_SMD:R_0603_1608Metric
- renumbered U2 to U1
Connections:
- net +5V is gone; now on net +3V3: J1.3 (P3)
- net +3V3: now also C1.1, D1.2 (C), D2.2 (C), D3.2 (C), J3.2 (P2), J3.6, J4.1 (VCC), R1.1, R10.2, R2.1; no longer U1.3 (EN)
- net GND: now also C1.2, D1.1 (A), D2.1 (A), D3.1 (A), J3.1 (P1), J3.7, J4.5 (GND)
- net SCL: now also J3.5 (P5), R10.1, R8.2; no longer U1.20 (GPIO5)
- net SDA: now also J3.4 (P4), R6.2; no longer U1.19 (GPIO4)
- net SENS: now also J3.3 (P3), R9.2; no longer U1.7 (GPIO13)
- net GPIO0: now reaches R3.1, U1.18 (GPIO0)
- net GPIO0: now also J4.2 (GPIO0)
- net RST: now reaches U1.1 (~{RST})
- net RST: now also J4.3 (~{RST}), R2.2
- net RX: now reaches U1.21 (GPIO3/RXD)
- net RX: now also J4.6 (RX)
- net TX: now reaches U1.22 (GPIO1/TXD)
- net TX: now also J4.4 (TX)
- new net: R1.2, U1.3 (EN)
- new net SCL_esp: D2.3 (C), R8.1, U1.20 (GPIO5)
- new net SDA_esp: D1.3 (C), R6.1, U1.19 (GPIO4)
- new net SENS_esp: D3.3 (C), R9.1, U1.7 (GPIO13)
- no-connect marks 16 -> 12
Other:
- note added: "GPIO0 -> 0 RST -> 0 -> 1"
- note added: "Protection"
- note removed: "Power source"
- title: LVL smart light + ESP8266 12-F -> LVL Light Control Board + ESP8266 - 12F
- moved on the sheet: J1, J2, R3, R4, R5, R7, U1

Commit message: BOM updated
Parts:
- R6, R8, R9: value R -> 220R
Changed lines of the file:
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@@
       (effects (font (size 1.27 1.27)))
     )
-    (property "Value" "R" (at 195.58 30.48 90)
+    (property "Value" "220R" (at 195.58 30.48 90)
       (effects (font (size 1.27 1.27)))
     )
@@
       (effects (font (size 1.27 1.27)))
     )
-    (property "Value" "R" (at 248.92 30.48 90)
+    (property "Value" "220R" (at 248.92 30.48 90)
       (effects (font (size 1.27 1.27)))
     )
@@
       (effects (font (size 1.27 1.27)))
     )
-    (property "Value" "R" (at 248.92 67.31 90)
-      (effects (font (size 1.27 1.27)))
-    )
+    (property "Value" "220R" (at 248.92 67.31 90)
+      (effects (font (size 1.27 1.27)))
+    )
